File: thermostat/sensors.sch (KiCad schematic (older format))
At the start: 12 parts, among them U2 MCP7940N-xMS, U3 MCP9844, U4 AT24C512, Y3 32.768KHz 20PPM 3.2x1.5mm 7PF

Commit message: Fine grouping of parts done, may start routing . GPIO connector on wrong side of PCB (I wanted to have the buttons on the opposite side, but thats not a big problem.
Parts:
- R5, R6: footprint Resistor_SMD:R_0603_1608Metric -> Resistor_SMD:R_0402_1005Metric
Changed lines of the file:
@@
 F 0 "R5" H 4570 5546 50  0000 L CNN
 F 1 "2k2" H 4570 5455 50  0000 L CNN
-F 2 "Resistor_SMD:R_0603_1608Metric" V 4430 5500 50  0001 C CNN
+F 2 "Resistor_SMD:R_0402_1005Metric" V 4430 5500 50  0001 C CNN
 F 3 "~" H 4500 5500 50  0001 C CNN
 	1    4500 5500
@@
 F 0 "R6" H 4920 5546 50  0000 L CNN
 F 1 "2k2" H 4920 5455 50  0000 L CNN
-F 2 "Resistor_SMD:R_0603_1608Metric" V 4780 5500 50  0001 C CNN
+F 2 "Resistor_SMD:R_0402_1005Metric" V 4780 5500 50  0001 C CNN
 F 3 "~" H 4850 5500 50  0001 C CNN
 	1    4850 5500

Commit message: Finished routing except for the RF line, still need to add many many grounding vias.
Parts:
- R5, R6: footprint Resistor_SMD:R_0402_1005Metric -> Resistor_SMD:R_0603_1608Metric
Changed lines of the file:
@@
 F 0 "R5" H 4570 5546 50  0000 L CNN
 F 1 "2k2" H 4570 5455 50  0000 L CNN
-F 2 "Resistor_SMD:R_0402_1005Metric" V 4430 5500 50  0001 C CNN
+F 2 "Resistor_SMD:R_0603_1608Metric" V 4430 5500 50  0001 C CNN
 F 3 "~" H 4500 5500 50  0001 C CNN
 	1    4500 5500
@@
 F 0 "R6" H 4920 5546 50  0000 L CNN
 F 1 "2k2" H 4920 5455 50  0000 L CNN
-F 2 "Resistor_SMD:R_0402_1005Metric" V 4780 5500 50  0001 C CNN
+F 2 "Resistor_SMD:R_0603_1608Metric" V 4780 5500 50  0001 C CNN
 F 3 "~" H 4850 5500 50  0001 C CNN
 	1    4850 5500
